File: bluetooth.sch (KiCad schematic (older format))
At the start: 4 parts

Commit message: Add bluetooth module lib
Parts:
- removed U?: MOUDLE-BLUETOOTH-HC-05(34P-27X13MM), BT34P-SMD-1.5-26.9X13.0X2.2MM, symbol MOUDLE-BLUETOOTH-HC-05(34P-27X13MM)
- added U?: MOUDLE-BLUETOOTH-HC-05(34P-27X13MM), BT34P-SMD-1.5-26.9X13.0X2.2MM, symbol MOUDLE-BLUETOOTH-HC-05(34P-27X13MM)
Connections:
- net +3V3: now also U?.12 (3.3V)
- net BLUETOOTH_RX: now also U?.2 (UART-RX)
- net BLUETOOTH_TX: now also U?.1 (UART-TX)
- net GND: now also U?.13 (GND0)
- net at J?.4 (P4): now also U?.16 (SPI_CSB)
- net at J?.3 (P3): now also U?.17 (SPI_MOSI)
- net at J?.2 (P2): now also U?.18 (SPI_MISO)
- net at J?.1 (P1): now also U?.19 (SPI_CLK)
Changed lines of the file:
@@
 LIBS:valves
 LIBS:stm32
-LIBS:MOUDLE-BLUETOOTH-HC-05_34P-27X13MM_
+LIBS:bluetooth_hc-05
 LIBS:smart_cutlery_pcb-cache
 EELAYER 25 0
@@
 Comment4 ""
 $EndDescr
-$Comp
-L MOUDLE-BLUETOOTH-HC-05(34P-27X13MM) U?
-U 1 1 599FE7A1
-P 5950 3100
-F 0 "U?" H 5050 3900 50  0000 L BNN
-F 1 "MOUDLE-BLUETOOTH-HC-05(34P-27X13MM)" H 5299 3901 50  0000 L BNN
-F 2 "BT34P-SMD-1.5-26.9X13.0X2.2MM" H 5950 3100 50  0001 L BNN
-F 3 "None" H 5950 3100 50  0001 L BNN
-F 4 "HC-05" H 5950 3100 50  0001 L BNN "MP"
-F 5 "SOIC-14 " H 5950 3100 50  0001 L BNN "Package"
-F 6 "Unavailable" H 5950 3100 50  0001 L BNN "Availability"
-F 7 "None" H 5950 3100 50  0001 L BNN "Description"
-F 8 "" H 5950 3100 50  0001 L BNN "MF"
-	1    5950 3100
-	1    0    0    -1
-$EndComp
 $Comp
 L +3.3V #PWR?
@@
 	3750 3450 3750 3500
 Connection ~ 3900 3450
+$Comp
+L MOUDLE-BLUETOOTH-HC-05(34P-27X13MM) U?
+U 1 1 59A0DEC9
+P 5950 3100
+F 0 "U?" H 5050 3900 50  0000 L BNN
+F 1 "MOUDLE-BLUETOOTH-HC-05(34P-27X13MM)" H 5299 3901 50  0000 L BNN
+F 2 "BT34P-SMD-1.5-26.9X13.0X2.2MM" H 5950 3100 50  0001 L BNN
+F 3 "None" H 5950 3100 50  0001 L BNN
+F 4 "HC-05" H 5950 3100 50  0001 L BNN "MP"
+F 5 "SOIC-14 " H 5950 3100 50  0001 L BNN "Package"
+F 6 "Unavailable" H 5950 3100 50  0001 L BNN "Availability"
+F 7 "None" H 5950 3100 50  0001 L BNN "Description"
+F 8 "" H 5950 3100 50  0001 L BNN "MF"
+	1    5950 3100
+	1    0    0    -1
+$EndComp
 $EndSCHEMATC

Commit message: Capture boost converter, soft latching power
Other:
- note added: "Firmware programming header"
Changed lines of the file:
@@
 LIBS:stm32
 LIBS:bluetooth_hc-05
+LIBS:mechanical
+LIBS:switches
+LIBS:NCP1402SN33T1G
+LIBS:diode
 LIBS:smart_cutlery_pcb-cache
 EELAYER 25 0
@@
 $Descr A4 11693 8268
 encoding utf-8
-Sheet 3 3
+Sheet 3 4
 Title ""
 Date ""
@@
 	1    0    0    -1
 $EndComp
+Text Notes 5400 4600 0    60   ~ 0
+Firmware programming header
 $EndSCHEMATC
