File: power.sch (KiCad schematic (older format))
At the start: 18 parts

Commit message: Add accelerometer/gyro
Connections:
- net BAT1_V: now reaches BT?.1 (+), D?.2 (A)
- net BAT2_V: now reaches BT?.1 (+), D?.2 (A)
Changed lines of the file:
@@
 LIBS:NCP1402SN33T1G
 LIBS:diode
+LIBS:battery_management
+LIBS:sensors
 LIBS:smart_cutlery_pcb-cache
 EELAYER 25 0
@@
 $Descr A4 11693 8268
 encoding utf-8
-Sheet 4 4
+Sheet 4 5
 Title ""
 Date ""
@@
 	1    0    0    -1
 $EndComp
+Wire Wire Line
+	2300 3750 2350 3750
+Connection ~ 2300 3750
+Wire Wire Line
+	1500 3750 1450 3750
+Connection ~ 1500 3750
+Text HLabel 1450 3750 0    60   Output ~ 0
+BAT1_V
+Text HLabel 2350 3750 2    60   Output ~ 0
+BAT2_V
 $EndSCHEMATC
