File: power.sch (KiCad schematic (older format))
At the start: 15 parts, among them Q1 BSS84, Q2 BSS138, SW1 TL3342, U3 NCP1402SN33T1G

Commit message: Update KiCAD version, add 150uH test, add text annotating component changes
Parts:
- Q2: symbol BSS138 -> BSS138-RESCUE-smart_cutlery_pcb
Other:
- note added: "0603 47uH <10% efficiency. Switched to 100uH, 30% efficiency"
- note added: "Currently testing different footprints..."
- note added: "FOR L2"
Changed lines of the file:
@@
 EESchema Schematic File Version 2
+LIBS:smart_cutlery_pcb-rescue
 LIBS:power
 LIBS:device
@@
 $EndComp
 $Comp
-L BSS138 Q2
+L BSS138-RESCUE-smart_cutlery_pcb Q2
 U 1 1 59AC415E
 P 3600 3900
+AR Path="/59AC415E" Ref="Q2"  Part="1"
+AR Path="/59A1225E/59AC415E" Ref="Q2"  Part="1"
 F 0 "Q2" H 3850 3950 50  0000 L CNN
 F 1 "BSS138" H 3800 3850 50  0000 L CNN
@@
 Connection ~ 4450 3000
 Connection ~ 4850 3950
+Text Notes 5000 1800 0    60   ~ 0
+0603 47uH <10% efficiency. Switched to 100uH, 30% efficiency
+Text Notes 5600 2000 0    60   ~ 0
+Currently testing different footprints...
+Text Notes 6300 1550 0    60   ~ 0
+FOR L2
 $EndSCHEMATC
