File: smart_cutlery_pcb.kicad_pcb (KiCad board)
At the start: 2 copper layers, 95 x 19.5 mm, 50 parts, among them J1 CONN_01X05, J2 CONN_01X04, Q1 BSS84, Q2 BSS138, SW1 TL3342, U1 STM32L053C6Tx, U2 MODULE-BLUETOOTH-HC-05(34P-27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, U3 NCP1402SN33T1G, U4 MPU-9250, U5 ASMT-YTC2-0AA02

Commit message: Place ref designators
Parts:
- added REF**: Measurement_Point_Square-SMD-Pad_Big, Measurement_Points:Measurement_Point_Square-SMD-Pad_Big, F.Cu at (108.8, 86.4)
- added REF**: Measurement_Point_Square-SMD-Pad_Big, Measurement_Points:Measurement_Point_Square-SMD-Pad_Big, F.Cu at (140.8, 94.4)
- added REF**: Measurement_Point_Square-SMD-Pad_Big, Measurement_Points:Measurement_Point_Square-SMD-Pad_Big, F.Cu at (108.8, 102.4)
- added REF**: Measurement_Point_Square-SMD-Pad_Big, Measurement_Points:Measurement_Point_Square-SMD-Pad_Big, F.Cu at (116.8, 102.4)
- added REF**: Measurement_Point_Square-SMD-Pad_Big, Measurement_Points:Measurement_Point_Square-SMD-Pad_Big, F.Cu at (124.8, 102.4)
- added REF**: Measurement_Point_Square-SMD-Pad_Big, Measurement_Points:Measurement_Point_Square-SMD-Pad_Big, F.Cu at (132.8, 102.4)
- added REF**: Measurement_Point_Square-SMD-Pad_Big, Measurement_Points:Measurement_Point_Square-SMD-Pad_Big, F.Cu at (140.8, 102.4)
- added REF**: Measurement_Point_Square-SMD-Pad_Big, Measurement_Points:Measurement_Point_Square-SMD-Pad_Big, F.Cu at (136.8, 106.5)
- added REF**: Measurement_Point_Square-SMD-Pad_Big, Measurement_Points:Measurement_Point_Square-SMD-Pad_Big, F.Cu at (128.8, 106.5)
- added REF**: Measurement_Point_Square-SMD-Pad_Big, Measurement_Points:Measurement_Point_Square-SMD-Pad_Big, F.Cu at (120.8, 106.5)
- added REF**: Measurement_Point_Square-SMD-Pad_Big, Measurement_Points:Measurement_Point_Square-SMD-Pad_Big, F.Cu at (112.8, 106.5)
- added REF**: Measurement_Point_Square-SMD-Pad_Big, Measurement_Points:Measurement_Point_Square-SMD-Pad_Big, F.Cu at (116.8, 86.4)
- added REF**: Measurement_Point_Square-SMD-Pad_Big, Measurement_Points:Measurement_Point_Square-SMD-Pad_Big, F.Cu at (104.8, 106.5)
- added REF**: Measurement_Point_Square-SMD-Pad_Big, Measurement_Points:Measurement_Point_Square-SMD-Pad_Big, F.Cu at (136.8, 98.5)
- added REF**: Measurement_Point_Square-SMD-Pad_Big, Measurement_Points:Measurement_Point_Square-SMD-Pad_Big, F.Cu at (128.8, 98.5)
- added REF**: Measurement_Point_Square-SMD-Pad_Big, Measurement_Points:Measurement_Point_Square-SMD-Pad_Big, F.Cu at (120.8, 98.5)
- added REF**: Measurement_Point_Square-SMD-Pad_Big, Measurement_Points:Measurement_Point_Square-SMD-Pad_Big, F.Cu at (112.8, 98.5)
- added REF**: Measurement_Point_Square-SMD-Pad_Big, Measurement_Points:Measurement_Point_Square-SMD-Pad_Big, F.Cu at (104.8, 98.5)
- added REF**: Measurement_Point_Square-SMD-Pad_Big, Measurement_Points:Measurement_Point_Square-SMD-Pad_Big, F.Cu at (136.8, 90.5)
- added REF**: Measurement_Point_Square-SMD-Pad_Big, Measurement_Points:Measurement_Point_Square-SMD-Pad_Big, F.Cu at (128.8, 90.5)
- added REF**: Measurement_Point_Square-SMD-Pad_Big, Measurement_Points:Measurement_Point_Square-SMD-Pad_Big, F.Cu at (120.8, 90.5)
- added REF**: Measurement_Point_Square-SMD-Pad_Big, Measurement_Points:Measurement_Point_Square-SMD-Pad_Big, F.Cu at (112.8, 90.5)
- added REF**: Measurement_Point_Square-SMD-Pad_Big, Measurement_Points:Measurement_Point_Square-SMD-Pad_Big, F.Cu at (124.8, 86.4)
- added REF**: Measurement_Point_Square-SMD-Pad_Big, Measurement_Points:Measurement_Point_Square-SMD-Pad_Big, F.Cu at (104.8, 90.5)
- added REF**: Measurement_Point_Square-SMD-Pad_Big, Measurement_Points:Measurement_Point_Square-SMD-Pad_Big, F.Cu at (132.8, 86.4)
- added REF**: Measurement_Point_Square-SMD-Pad_Big, Measurement_Points:Measurement_Point_Square-SMD-Pad_Big, F.Cu at (140.8, 86.4)
- added REF**: Measurement_Point_Square-SMD-Pad_Big, Measurement_Points:Measurement_Point_Square-SMD-Pad_Big, F.Cu at (108.8, 94.4)
- added REF**: Measurement_Point_Square-SMD-Pad_Big, Measurement_Points:Measurement_Point_Square-SMD-Pad_Big, F.Cu at (116.8, 94.4)
- added REF**: Measurement_Point_Square-SMD-Pad_Big, Measurement_Points:Measurement_Point_Square-SMD-Pad_Big, F.Cu at (124.8, 94.4)
- added REF**: Measurement_Point_Square-SMD-Pad_Big, Measurement_Points:Measurement_Point_Square-SMD-Pad_Big, F.Cu at (132.8, 94.4)
