File: micro.sch (KiCad schematic (older format))
At the start: 12 parts

Commit message: Make top-level connections between microcontroller and everything else
Parts:
- gave numbers to parts that had none: 12
Changed lines of the file:
@@
 $EndDescr
 $Comp
-L STM32L053C6Tx U?
+L STM32L053C6Tx U1
 U 1 1 599E9E22
 P 5800 3800
-F 0 "U?" H 2200 5625 50  0000 L BNN
+F 0 "U1" H 2200 5625 50  0000 L BNN
 F 1 "STM32L053C6Tx" H 9400 5625 50  0000 R BNN
 F 2 "Housings_QFP:LQFP-48_7x7mm_Pitch0.5mm" H 9400 5575 50  0001 R TNN
@@
 PB15
 $Comp
-L +3.3V #PWR?
+L +3.3V #PWR01
 U 1 1 599F30E1
 P 5600 1300
-F 0 "#PWR?" H 5600 1150 50  0001 C CNN
+F 0 "#PWR01" H 5600 1150 50  0001 C CNN
 F 1 "+3.3V" H 5600 1440 50  0000 C CNN
 F 2 "" H 5600 1300 50  0001 C CNN
@@
 $EndComp
 $Comp
-L GND #PWR?
+L GND #PWR02
 U 1 1 599F32B0
 P 5600 5900
-F 0 "#PWR?" H 5600 5650 50  0001 C CNN
+F 0 "#PWR02" H 5600 5650 50  0001 C CNN
 F 1 "GND" H 5600 5750 50  0000 C CNN
 F 2 "" H 5600 5900 50  0001 C CNN
@@
 $EndComp
 $Comp
-L L_Small L?
+L L_Small L1
 U 1 1 599F364C
 P 6250 1350
-F 0 "L?" V 6350 1300 50  0000 L CNN
+F 0 "L1" V 6350 1300 50  0000 L CNN
 F 1 "Ferrite" V 6200 1200 50  0000 L CNN
 F 2 "" H 6250 1350 50  0001 C CNN
@@
 $EndComp
 $Comp
-L C_Small C?
+L C_Small C5
 U 1 1 599F37D8
 P 6900 1450
-F 0 "C?" H 6910 1520 50  0000 L CNN
+F 0 "C5" H 6910 1520 50  0000 L CNN
 F 1 "100n" H 6700 1400 50  0000 L CNN
 F 2 "" H 6900 1450 50  0001 C CNN
@@
 $EndComp
 $Comp
-L C_Small C?
+L C_Small C6
 U 1 1 599F38C9
 P 7200 1450
-F 0 "C?" H 7210 1520 50  0000 L CNN
+F 0 "C6" H 7210 1520 50  0000 L CNN
 F 1 "1uF" H 7250 1400 50  0000 L CNN
 F 2 "" H 7200 1450 50  0001 C CNN
@@
 $EndComp
 $Comp
-L GND #PWR?
+L GND #PWR03
 U 1 1 599F39C8
 P 7050 1600
-F 0 "#PWR?" H 7050 1350 50  0001 C CNN
+F 0 "#PWR03" H 7050 1350 50  0001 C CNN
 F 1 "GND" H 7050 1450 50  0000 C CNN
 F 2 "" H 7050 1600 50  0001 C CNN
@@
 $EndComp
 $Comp
-L C_Small C?
+L C_Small C3
 U 1 1 599F4030
 P 4650 1350
-F 0 "C?" H 4660 1420 50  0000 L CNN
+F 0 "C3" H 4660 1420 50  0000 L CNN
 F 1 "100n" H 4450 1300 50  0000 L CNN
 F 2 "" H 4650 1350 50  0001 C CNN
@@
 $EndComp
 $Comp
-L C_Small C?
+L C_Small C4
 U 1 1 599F409F
 P 4950 1350
-F 0 "C?" H 4960 1420 50  0000 L CNN
+F 0 "C4" H 4960 1420 50  0000 L CNN
 F 1 "1uF" H 4750 1300 50  0000 L CNN
 F 2 "" H 4950 1350 50  0001 C CNN
@@
 $EndComp
 $Comp
-L C_Small C?
+L C_Small C2
 U 1 1 599F4143
 P 4350 1350
-F 0 "C?" H 4360 1420 50  0000 L CNN
+F 0 "C2" H 4360 1420 50  0000 L CNN
 F 1 "100n" H 4150 1300 50  0000 L CNN
 F 2 "" H 4350 1350 50  0001 C CNN
@@
 $EndComp
 $Comp
-L C_Small C?
+L C_Small C1
 U 1 1 599F4178
 P 4050 1350
-F 0 "C?" H 4060 1420 50  0000 L CNN
+F 0 "C1" H 4060 1420 50  0000 L CNN
 F 1 "100n" H 3850 1300 50  0000 L CNN
 F 2 "" H 4050 1350 50  0001 C CNN
@@
 $EndComp
 $Comp
-L +3.3V #PWR?
+L +3.3V #PWR04
 U 1 1 599F41A8
 P 4050 1150
-F 0 "#PWR?" H 4050 1000 50  0001 C CNN
+F 0 "#PWR04" H 4050 1000 50  0001 C CNN
 F 1 "+3.3V" H 4050 1290 50  0000 C CNN
 F 2 "" H 4050 1150 50  0001 C CNN
@@
 $EndComp
 $Comp
-L GND #PWR?
+L GND #PWR05
 U 1 1 599F41CB
 P 4050 1550
-F 0 "#PWR?" H 4050 1300 50  0001 C CNN
+F 0 "#PWR05" H 4050 1300 50  0001 C CNN
 F 1 "GND" H 4050 1400 50  0000 C CNN
 F 2 "" H 4050 1550 50  0001 C CNN
@@
 Clean up the analog VDD a bit (because of touch stuff)
 $Comp
-L R R?
+L R R1
 U 1 1 599F721F
 P 1500 2700
-F 0 "R?" V 1580 2700 50  0000 C CNN
+F 0 "R1" V 1580 2700 50  0000 C CNN
 F 1 "4.7k" V 1500 2700 50  0000 C CNN
 F 2 "" V 1430 2700 50  0001 C CNN
@@
 $EndComp
 $Comp
-L GND #PWR?
+L GND #PWR06
 U 1 1 599F73E8
 P 1350 2700
-F 0 "#PWR?" H 1350 2450 50  0001 C CNN
+F 0 "#PWR06" H 1350 2450 50  0001 C CNN
 F 1 "GND" H 1350 2550 50  0000 C CNN
 F 2 "" H 1350 2700 50  0001 C CNN
@@
 $EndComp
 $Comp
-L +3.3V #PWR?
+L +3.3V #PWR07
 U 1 1 599F7696
 P 2100 2900
-F 0 "#PWR?" H 2100 2750 50  0001 C CNN
+F 0 "#PWR07" H 2100 2750 50  0001 C CNN
 F 1 "+3.3V" H 2100 3040 50  0000 C CNN
 F 2 "" H 2100 2900 50  0001 C CNN
@@
 SWD_CLK
 $Comp
-L CONN_01X05 J?
+L CONN_01X05 J1
 U 1 1 599F8D75
 P 10500 1450
-F 0 "J?" H 10500 1750 50  0000 C CNN
+F 0 "J1" H 10500 1750 50  0000 C CNN
 F 1 "CONN_01X05" V 10600 1450 50  0000 C CNN
 F 2 "" H 10500 1450 50  0001 C CNN
@@
 SWD_CLK
 $Comp
-L +3.3V #PWR?
+L +3.3V #PWR08
 U 1 1 599FA6C7
 P 9300 1250
-F 0 "#PWR?" H 9300 1100 50  0001 C CNN
+F 0 "#PWR08" H 9300 1100 50  0001 C CNN
 F 1 "+3.3V" H 9300 1390 50  0000 C CNN
 F 2 "" H 9300 1250 50  0001 C CNN
@@
 $EndComp
 $Comp
-L GND #PWR?
+L GND #PWR09
 U 1 1 599FA920
 P 9300 1450
-F 0 "#PWR?" H 9300 1200 50  0001 C CNN
+F 0 "#PWR09" H 9300 1200 50  0001 C CNN
 F 1 "GND" H 9300 1300 50  0000 C CNN
 F 2 "" H 9300 1450 50  0001 C CNN
@@
 $EndComp
 $Comp
-L R R?
+L R R3
 U 1 1 599FAFFB
 P 10100 1550
-F 0 "R?" V 10180 1550 50  0000 C CNN
+F 0 "R3" V 10180 1550 50  0000 C CNN
 F 1 "100" V 10100 1550 50  0000 C CNN
 F 2 "" V 10030 1550 50  0001 C CNN
@@
 $EndComp
 $Comp
-L R R?
+L R R2
 U 1 1 599FB16D
 P 10100 1350
-F 0 "R?" V 10180 1350 50  0000 C CNN
+F 0 "R2" V 10180 1350 50  0000 C CNN
 F 1 "100" V 10100 1350 50  0000 C CNN
 F 2 "" V 10030 1350 50  0001 C CNN

Commit message: Assigned some footprints and added CR1225 holder footprint
Parts:
- C1, C2, C3, C4, C5, C6: footprint (none) -> Capacitors_SMD:C_0603
- J1: footprint (none) -> Pin_Headers:Pin_Header_Straight_1x05_Pitch2.54mm
- R1, R2, R3: footprint (none) -> Resistors_SMD:R_0603
Changed lines of the file:
@@
 F 0 "C5" H 6910 1520 50  0000 L CNN
 F 1 "100n" H 6700 1400 50  0000 L CNN
-F 2 "" H 6900 1450 50  0001 C CNN
+F 2 "Capacitors_SMD:C_0603" H 6900 1450 50  0001 C CNN
 F 3 "" H 6900 1450 50  0001 C CNN
 	1    6900 1450
@@
 F 0 "C6" H 7210 1520 50  0000 L CNN
 F 1 "1uF" H 7250 1400 50  0000 L CNN
-F 2 "" H 7200 1450 50  0001 C CNN
+F 2 "Capacitors_SMD:C_0603" H 7200 1450 50  0001 C CNN
 F 3 "" H 7200 1450 50  0001 C CNN
 	1    7200 1450
@@
 F 0 "C3" H 4660 1420 50  0000 L CNN
 F 1 "100n" H 4450 1300 50  0000 L CNN
-F 2 "" H 4650 1350 50  0001 C CNN
+F 2 "Capacitors_SMD:C_0603" H 4650 1350 50  0001 C CNN
 F 3 "" H 4650 1350 50  0001 C CNN
 	1    4650 1350
@@
 F 0 "C4" H 4960 1420 50  0000 L CNN
 F 1 "1uF" H 4750 1300 50  0000 L CNN
-F 2 "" H 4950 1350 50  0001 C CNN
+F 2 "Capacitors_SMD:C_0603" H 4950 1350 50  0001 C CNN
 F 3 "" H 4950 1350 50  0001 C CNN
 	1    4950 1350
@@
 F 0 "C2" H 4360 1420 50  0000 L CNN
 F 1 "100n" H 4150 1300 50  0000 L CNN
-F 2 "" H 4350 1350 50  0001 C CNN
+F 2 "Capacitors_SMD:C_0603" H 4350 1350 50  0001 C CNN
 F 3 "" H 4350 1350 50  0001 C CNN
 	1    4350 1350
@@
 F 0 "C1" H 4060 1420 50  0000 L CNN
 F 1 "100n" H 3850 1300 50  0000 L CNN
-F 2 "" H 4050 1350 50  0001 C CNN
+F 2 "Capacitors_SMD:C_0603" H 4050 1350 50  0001 C CNN
 F 3 "" H 4050 1350 50  0001 C CNN
 	1    4050 1350
@@
 F 0 "R1" V 1580 2700 50  0000 C CNN
 F 1 "4.7k" V 1500 2700 50  0000 C CNN
-F 2 "" V 1430 2700 50  0001 C CNN
+F 2 "Resistors_SMD:R_0603" V 1430 2700 50  0001 C CNN
 F 3 "" H 1500 2700 50  0001 C CNN
 	1    1500 2700
@@
 F 0 "J1" H 10500 1750 50  0000 C CNN
 F 1 "CONN_01X05" V 10600 1450 50  0000 C CNN
-F 2 "" H 10500 1450 50  0001 C CNN
+F 2 "Pin_Headers:Pin_Header_Straight_1x05_Pitch2.54mm" H 10500 1450 50  0001 C CNN
 F 3 "" H 10500 1450 50  0001 C CNN
 	1    10500 1450
@@
 F 0 "R3" V 10180 1550 50  0000 C CNN
 F 1 "100" V 10100 1550 50  0000 C CNN
-F 2 "" V 10030 1550 50  0001 C CNN
+F 2 "Resistors_SMD:R_0603" V 10030 1550 50  0001 C CNN
 F 3 "" H 10100 1550 50  0001 C CNN
 	1    10100 1550
@@
 F 0 "R2" V 10180 1350 50  0000 C CNN
 F 1 "100" V 10100 1350 50  0000 C CNN
-F 2 "" V 10030 1350 50  0001 C CNN
+F 2 "Resistors_SMD:R_0603" V 10030 1350 50  0001 C CNN
 F 3 "" H 10100 1350 50  0001 C CNN
 	1    10100 1350

Commit message: Add switch footprints, add mode switch
Parts:
- L1: footprint (none) -> Inductors_SMD:L_0603
Changed lines of the file:
@@
 F 0 "L1" V 6350 1300 50  0000 L CNN
 F 1 "Ferrite" V 6200 1200 50  0000 L CNN
-F 2 "" H 6250 1350 50  0001 C CNN
+F 2 "Inductors_SMD:L_0603" H 6250 1350 50  0001 C CNN
 F 3 "" H 6250 1350 50  0001 C CNN
 	1    6250 1350

Commit message: More changes, replace
Parts:
- removed C4, C6: 1uF, Capacitors_SMD:C_0603, symbol C_Small
Changed lines of the file:
@@
-$EndComp
-$Comp
-L C_Small C6
-U 1 1 599F38C9
-P 7200 1450
-F 0 "C6" H 7210 1520 50  0000 L CNN
-F 1 "1uF" H 7250 1400 50  0000 L CNN
-F 2 "Capacitors_SMD:C_0603" H 7200 1450 50  0001 C CNN
-F 3 "" H 7200 1450 50  0001 C CNN
-	1    7200 1450
-	1    0    0    -1
 $EndComp
 $Comp
 L GND #PWR03
 U 1 1 599F39C8
-P 7050 1600
-F 0 "#PWR03" H 7050 1350 50  0001 C CNN
-F 1 "GND" H 7050 1450 50  0000 C CNN
-F 2 "" H 7050 1600 50  0001 C CNN
-F 3 "" H 7050 1600 50  0001 C CNN
-	1    7050 1600
+P 6900 1550
+F 0 "#PWR03" H 6900 1300 50  0001 C CNN
+F 1 "GND" H 6900 1400 50  0000 C CNN
+F 2 "" H 6900 1550 50  0001 C CNN
+F 3 "" H 6900 1550 50  0001 C CNN
+	1    6900 1550
 	1    0    0    -1
 $EndComp
@@
 F 3 "" H 4650 1350 50  0001 C CNN
 	1    4650 1350
-	1    0    0    -1
-$EndComp
-$Comp
-L C_Small C4
-U 1 1 599F409F
-P 4950 1350
-F 0 "C4" H 4960 1420 50  0000 L CNN
-F 1 "1uF" H 4750 1300 50  0000 L CNN
-F 2 "Capacitors_SMD:C_0603" H 4950 1350 50  0001 C CNN
-F 3 "" H 4950 1350 50  0001 C CNN
-	1    4950 1350
 	1    0    0    -1
 $EndComp
@@
 Wire Wire Line
 	6750 1450 6750 1350
-Wire Wire Line
-	6350 1350 7200 1350
 Connection ~ 6750 1350
 Connection ~ 6900 1350
@@
 Connection ~ 5600 1350
 Wire Wire Line
-	6900 1550 7200 1550
-Wire Wire Line
-	7050 1600 7050 1550
-Connection ~ 7050 1550
-Wire Wire Line
 	4050 1450 4050 1550
-Wire Wire Line
-	4050 1500 4950 1500
-Wire Wire Line
-	4950 1500 4950 1450
 Wire Wire Line
 	4650 1450 4650 1500
@@
 Wire Wire Line
 	4050 1150 4050 1250
-Wire Wire Line
-	4050 1200 4950 1200
-Wire Wire Line
-	4950 1200 4950 1250
 Wire Wire Line
 	4350 1250 4350 1200
@@
 Text Notes 750  3500 0    60   ~ 0
 These pins were for\noscillators. Can meb\nbe used as GPIOS\nbut meh.
+Wire Wire Line
+	6350 1350 6900 1350
+Wire Wire Line
+	4650 1200 4050 1200
+Wire Wire Line
+	4650 1500 4050 1500
 $EndSCHEMATC

Commit message: Create relevant BOM links, export digikey BOM
Parts:
- L1: value Ferrite -> 47uH; MFR (none) -> Taiyo Yuden; MPN (none) -> CBMF1608T470K; SPN (none) -> 587-1722-1-ND; SPR (none) -> https://www.digikey.com.au/
- U1: MFR (none) -> STMicroelectronics; MPN (none) -> STM32L053C8T6; SPN (none) -> 497-14906-ND; SPR (none) -> https://www.digikey.com.au/
